Commit message: update the dragon model for valve manipulate

File: dragon_valve/urdf/dragon.urdf.xacro (robot description, xacro)
@@ -3,23 +3,21 @@
     xmlns:xacro="http://www.ros.org/wiki/xacro" name="dragon" >
   <xacro:include filename="$(find dragon)/robots/quad/euclid_201709.urdf.xacro" />
+  <xacro:property name="offset" value="0.013" />
   <joint name="gripper_joint" type="fixed">
     <parent link="link1"/>
     <child link="gripper"/>
-    <origin rpy="0 0 ${pi}" xyz="0.01 0.0 0"/>
+    <origin xyz="${offset} 0 0" rpy="0 0 ${pi}"/>
     <axis xyz="0 0 1"/>
   </joint>
   <link name="gripper">
-    <!-- <visual> -->
-    <!--   <origin xyz="0 0 0" rpy="0 0 0" /> -->
-    <!--   <geometry> -->
-    <!--     <sphere radius="0.033" /> -->
-    <!--   </geometry> -->
-    <!--   <material name="Yellow"> -->
-    <!--     <color rgba="1.0 1.0 0 1.0"/> -->
-    <!--   </material> -->
-    <!-- </visual> -->
+    <visual>
+      <origin xyz="-${offset} 0 0" rpy="0 0 0"/>
+      <geometry>
+        <mesh filename="package://dragon_valve/urdf/mesh/valve_gripper.dae"/>
+      </geometry>
+    </visual>
     <inertial>
-      <origin xyz="0 0 0" rpy="0 0 0"/>
-      <mass value="0.05"/>
+      <origin xyz="-${offset} 0 0" rpy="0 0 0"/>
+      <mass value="${0.0856 - 0.0452}"/> <!-- additional weight compared to stantdard gripper  -->
       <inertia
           ixx="0.00001" ixy="0.0" ixz="0.0"

Commit message: Add valve gazebo model and tip collision to enable valve manipulation in simulation

File: dragon_valve/urdf/dragon.urdf.xacro (robot description, xacro)
@@ -26,3 +26,31 @@
     </inertial>
   </link>
+  <joint name="tip1_joint" type="fixed">
+    <parent link="gripper"/>
+    <child link="tip1"/>
+    <origin xyz="0 0 0.07" rpy="0 0 0"/>
+    <axis xyz="0 0 1"/>
+  </joint>
+  <link name="tip1">
+    <collision>
+      <origin xyz="0.05 0 0" rpy="0 ${pi/2} 0"/>
+      <geometry>
+        <cylinder length="0.1" radius="0.006"/>
+      </geometry>
+    </collision>
+  </link>
+  <joint name="tip2_joint" type="fixed">
+    <parent link="gripper"/>
+    <child link="tip2"/>
+    <origin xyz="0 0 -0.07" rpy="0 0 0"/>
+    <axis xyz="0 0 1"/>
+  </joint>
+  <link name="tip2">
+    <collision>
+      <origin xyz="0.05 0 0" rpy="0 ${pi/2} 0"/>
+      <geometry>
+        <cylinder length="0.1" radius="0.006"/>
+      </geometry>
+    </collision>
+  </link>
 </robot>
