Commit message: Improve the valve model in urdf

File: dragon_valve/urdf/valve.urdf (robot description, URDF)
Before this commit: robot valve, 3 links, 2 joints
Links:
- removed link base
- removed link stem
Joints:
- added joint pipe_joint1: type fixed, parent main_pipe, child sub_pipe1, origin xyz=0 ${main_pipe_length * 0.5 - pipe_radius} 0 rpy=0 0 0, axis 0 0 1
- added joint pipe_joint2: type fixed, parent main_pipe, child sub_pipe2, origin xyz=0 -${main_pipe_length * 0.5 - pipe_radius} 0 rpy=0 0 0, axis 0 0 1
- added joint valve_pipe_joint: type fixed, parent main_pipe, child valve, origin xyz=0 0 ${valve_height} rpy=0 ${ $(arg valve_pitch_angle) / 180 * pi} 0, axis 0 0 1
- joint stem_joint: origin xyz=0 0 ${valve_height} rpy=0 0 0 -> xyz=0 0 ${pipe_radius * 2} rpy=0 0 0; parent base -> valve

Commit message: Add no collsion model for valve urdf model

File: dragon_valve/urdf/valve.urdf (robot description, URDF)
Before this commit: robot valve, 1 links, 5 joints
Links:
- link handle: geometry visual mesh filename=package://dragon_valve/urdf/mesh/200mm_valve.STL scale=0.001 0.001 0.001
